Commit message: fix wheel robot

File: totem/bot/urdf/bot.urdf.xacro (robot description, xacro)
@@ -32,5 +32,4 @@
 	<link name="back_left_wheel">
   		<visual>
-		    <origin xyz="1.24 -1.45 -0.07" rpy="0 1.57 0"/>
 			<geometry>
 				<cylinder radius="0.5" length="0.2"/>
@@ -43,5 +42,4 @@
 	<link name="back_right_wheel">
   		<visual>
-		    <origin xyz="-1.24 -1.45 -0.07" rpy="0 1.57 0"/>
 			<geometry>
 				<cylinder radius="0.5" length="0.2"/>
@@ -54,5 +52,4 @@
 	<link name="front_left_wheel">
   		<visual>
-		    <origin xyz="1.24 1.45 -0.07" rpy="0 1.57 0"/>
 			<geometry>
 				<cylinder radius="0.5" length="0.2"/>
@@ -65,5 +62,4 @@
 	<link name="front_right_wheel">
   		<visual>
-		    <origin xyz="-1.24 1.45 -0.07" rpy="0 1.57 0"/>
 			<geometry>
 				<cylinder radius="0.5" length="0.2"/>
@@ -108,4 +104,5 @@
   	</link>
 	<joint name="front_right_joint" type="continuous">
+		<origin xyz="-1.24 1.45 -0.07" rpy="0 1.57 0"/>
         <parent link="base_link"/>
         <child link="front_right_wheel"/>
@@ -115,4 +112,5 @@
  	</joint>
 	<joint name="front_left_joint" type="continuous">
+		<origin xyz="1.24 1.45 -0.07" rpy="0 1.57 0"/>
         <parent link="base_link"/>
         <child link="front_left_wheel"/>
@@ -121,4 +119,5 @@
  	</joint>
 	<joint name="back_right_joint" type="continuous">
+		<origin xyz="-1.24 -1.45 -0.07" rpy="0 1.57 0"/>
         <parent link="base_link"/>
         <child link="back_right_wheel"/>
@@ -127,4 +126,5 @@
  	</joint>
 	<joint name="back_left_joint" type="continuous">
+		<origin xyz="1.24 -1.45 -0.07" rpy="0 1.57 0"/>
         <parent link="base_link"/>
         <child link="back_left_wheel"/>

Commit message: new fix wheels

File: totem/bot/urdf/bot.urdf.xacro (robot description, xacro)
@@ -32,4 +32,5 @@
 	<link name="back_left_wheel">
   		<visual>
+		    <origin xyz="0 0 0" rpy="0 0 0"/>
 			<geometry>
 				<cylinder radius="0.5" length="0.2"/>
@@ -42,4 +43,5 @@
 	<link name="back_right_wheel">
   		<visual>
+		    <origin xyz="0 0 0" rpy="0 0 0"/>
 			<geometry>
 				<cylinder radius="0.5" length="0.2"/>
@@ -52,4 +54,5 @@
 	<link name="front_left_wheel">
   		<visual>
+		    <origin xyz="0 0 0" rpy="0 0 0"/>
 			<geometry>
 				<cylinder radius="0.5" length="0.2"/>
@@ -62,4 +65,5 @@
 	<link name="front_right_wheel">
   		<visual>
+		    <origin xyz="0 0 0" rpy="0 0 0"/>
 			<geometry>
 				<cylinder radius="0.5" length="0.2"/>
@@ -108,5 +112,5 @@
         <child link="front_right_wheel"/>
 		<limit effort="30" velocity="2.0"/>
-      	<axis xyz="1 0 0" />
+      	<axis xyz="0 0 1" />
       	<dynamics damping="1.0" />
  	</joint>
@@ -115,5 +119,5 @@
         <parent link="base_link"/>
         <child link="front_left_wheel"/>
-		<axis xyz="1 0 0"/>
+		<axis xyz="0 0 1"/>
 		<limit effort="30" velocity="2.0"/>
  	</joint>
@@ -122,5 +126,5 @@
         <parent link="base_link"/>
         <child link="back_right_wheel"/>
-		<axis xyz="1 0 0"/>
+		<axis xyz="0 0 1"/>
 		<limit effort="30" velocity="2.0"/>
  	</joint>
@@ -129,5 +133,5 @@
         <parent link="base_link"/>
         <child link="back_left_wheel"/>
-		<axis xyz="1 0 0"/>
+		<axis xyz="0 0 1"/>
 		<limit effort="30" velocity="2.0"/>
  	</joint>

Commit message: fixing urdf collision and inertia

File: totem/bot/urdf/bot.urdf.xacro (robot description, xacro)
@@ -2,4 +2,9 @@
 <robot name="bot">
  	<link name="base_link">
+	    <inertial>
+			<!-- <origin xyz="0 0 0.5" rpy="0 0 0"/> -->
+			<mass value="1"/>
+			<inertia ixx="2.3" ixy="0" ixz="0" iyy="3.35" iyz="0.00" izz="1.22" />
+		</inertial>
 		<visual>
 		    <origin xyz="1.05 0 0" rpy="0 0 0"/>
@@ -29,50 +34,113 @@
 	     	</material>
 		</visual>
+		<collision>
+		    <origin xyz="0 -1.95 0" rpy="0 0 0"/>
+			<geometry>
+				<box size="2 0.1 1"/>
+			</geometry>
+		</collision>
+		<collision>
+		    <origin xyz="1.05 0 0" rpy="0 0 0"/>
+			<geometry>
+				<box size="0.1 4 1"/>
+			</geometry>
+		</collision>
+		<collision>
+		    <origin xyz="-1.05 0 0" rpy="0 0 0"/>
+			<geometry>
+				<box size="0.1 4 1"/>
+			</geometry>
+		</collision>
   	</link>
 	<link name="back_left_wheel">
-  		<visual>
-		    <origin xyz="0 0 0" rpy="0 0 0"/>
-			<geometry>
-				<cylinder radius="0.5" length="0.2"/>
-			</geometry>
-			<material name="d">
-	       		<color rgba="0 0 0 0"/>
-	     	</material>
-		</visual>
+		<inertial>
+			<mass value="100"/>
+			<inertia ixx="0.2" ixy="0" ixz="0" iyy="0.2" iyz="0" izz="0.2"/>
+		</inertial>
+  		<visual>
+		    <origin xyz="0 0 0" rpy="0 0 0"/>
+			<geometry>
+				<cylinder radius="0.5" length="0.2"/>
+			</geometry>
+			<material name="d">
+	       		<color rgba="0 0 0 0"/>
+	     	</material>
+		</visual>
+		<collision>
+		    <origin xyz="0 0 0" rpy="0 0 0"/>
+			<geometry>
+				<cylinder radius="0.5" length="0.2"/>
+			</geometry>
+		</collision>
   	</link>
 	<link name="back_right_wheel">
-  		<visual>
-		    <origin xyz="0 0 0" rpy="0 0 0"/>
-			<geometry>
-				<cylinder radius="0.5" length="0.2"/>
-			</geometry>
-			<material name="d">
-	       		<color rgba="0 0 0 0"/>
-	     	</material>
-		</visual>
+		<inertial>
+			<mass value="100"/>
+			<inertia ixx="0.2" ixy="0" ixz="0" iyy="0.2" iyz="0" izz="0.2"/>
+		</inertial>
+  		<visual>
+		    <origin xyz="0 0 0" rpy="0 0 0"/>
+			<geometry>
+				<cylinder radius="0.5" length="0.2"/>
+			</geometry>
+			<material name="d">
+	       		<color rgba="0 0 0 0"/>
+	     	</material>
+		</visual>
+		<collision>
+		    <origin xyz="0 0 0" rpy="0 0 0"/>
+			<geometry>
+				<cylinder radius="0.5" length="0.2"/>
+			</geometry>
+		</collision>
   	</link>
 	<link name="front_left_wheel">
-  		<visual>
-		    <origin xyz="0 0 0" rpy="0 0 0"/>
-			<geometry>
-				<cylinder radius="0.5" length="0.2"/>
-			</geometry>
-			<material name="d">
-	       		<color rgba="0 0 0 0"/>
-	     	</material>
-		</visual>
+		<inertial>
+			<mass value="100"/>
+			<inertia ixx="0.2" ixy="0" ixz="0" iyy="0.2" iyz="0" izz="0.2"/>
+		</inertial>
+  		<visual>
+		    <origin xyz="0 0 0" rpy="0 0 0"/>
+			<geometry>
+				<cylinder radius="0.5" length="0.2"/>
+			</geometry>
+			<material name="d">
+	       		<color rgba="0 0 0 0"/>
+	     	</material>
+		</visual>
+		<collision>
+		    <origin xyz="0 0 0" rpy="0 0 0"/>
+			<geometry>
+				<cylinder radius="0.5" length="0.2"/>
+			</geometry>
+		</collision>
   	</link>
 	<link name="front_right_wheel">
-  		<visual>
-		    <origin xyz="0 0 0" rpy="0 0 0"/>
-			<geometry>
-				<cylinder radius="0.5" length="0.2"/>
-			</geometry>
-			<material name="d">
-	       		<color rgba="0 0 0 0"/>
-	     	</material>
-		</visual>
+		<inertial>
+			<mass value="100"/>
+			<inertia ixx="0.2" ixy="0" ixz="0" iyy="0.2" iyz="0" izz="0.2"/>
+		</inertial>
+  		<visual>
+		    <origin xyz="0 0 0" rpy="0 0 0"/>
+			<geometry>
+				<cylinder radius="0.5" length="0.2"/>
+			</geometry>
+			<material name="d">
+	       		<color rgba="0 0 0 0"/>
+	     	</material>
+		</visual>
+		<collision>
+		    <origin xyz="0 0 0" rpy="0 0 0"/>
+			<geometry>
+				<cylinder radius="0.5" length="0.2"/>
+			</geometry>
+		</collision>
   	</link>
 	<link name="front_panel">
+		<inertial>
+			<origin xyz="0 1.95 0" rpy="0 0 0"/>
+			<mass value="100"/>
+			<inertia ixx="0.2" ixy="0" ixz="0" iyy="0.2" iyz="0" izz="0.2"/>
+		</inertial>
   		<visual>
 		    <origin xyz="0 1.95 0" rpy="0 0 0"/>
@@ -84,4 +152,10 @@
 	     	</material>
 		</visual>
+		<collision>
+		    <origin xyz="0 1.95 0" rpy="0 0 0"/>
+			<geometry>
+				<box size="2 0.1 1"/>
+			</geometry>
+		</collision>
   	</link>
 	<link name="mid_panel">
@@ -95,4 +169,10 @@
 	     	</material>
 		</visual>
+		<collision>
+		    <origin xyz="0 0 0" rpy="0 0 0"/>
+			<geometry>
+				<box size="1.9 0.02 1"/>
+			</geometry>
+		</collision>
   	</link>
 	<link name="mid_panel_prism">

Commit message: correction urdf, ajout des collisions et des inerties, affichage fonctionnelle sur gazebo

File: totem/bot/urdf/bot.urdf.xacro (robot description, xacro)
@@ -1,10 +1,33 @@
 <?xml version="1.0"?>
-<robot name="bot">
+<robot name="bot" xmlns:xacro="http://ros.org/wiki/xacro">
+	<!-- Define intertial property macros  -->
+	<xacro:macro name="box_inertia" params="m w h d">
+		<inertial>
+		<origin xyz="0 0 0" rpy="${pi/2} 0 ${pi/2}"/>
+		<mass value="${m}"/>
+		<inertia ixx="${(m/12) * (h*h + d*d)}" ixy="0.0" ixz="0.0" iyy="${(m/12) * (w*w + d*d)}" iyz="0.0" izz="${(m/12) * (w*w + h*h)}"/>
+		</inertial>
+	</xacro:macro>
+	<xacro:macro name="cylinder_inertia" params="m r h">
+		<inertial>
+		<origin xyz="0 0 0" rpy="${pi/2} 0 0" />
+		<mass value="${m}"/>
+		<inertia ixx="${(m/12) * (3*r*r + h*h)}" ixy = "0" ixz = "0" iyy="${(m/12) * (3*r*r + h*h)}" iyz = "0" izz="${(m/2) * (r*r)}"/>
+		</inertial>
+	</xacro:macro>
+	<xacro:macro name="sphere_inertia" params="m r">
+		<inertial>
+		<mass value="${m}"/>
+		<inertia ixx="${(2/5) * m * (r*r)}" ixy="0.0" ixz="0.0" iyy="${(2/5) * m * (r*r)}" iyz="0.0" izz="${(2/5) * m * (r*r)}"/>
+		</inertial>
+	</xacro:macro>
+	<link name="base_footprint"/>
+	<!-- The base footprint of the robot is located underneath the chassis -->
+	<joint name="base_joint" type="fixed">
+		<parent link="base_link"/>
+		<child link="base_footprint" />
+		<origin xyz="0.0 0.0 -0.1" rpy="0 0 0"/>
+	</joint>
  	<link name="base_link">
-	    <inertial>
-			<!-- <origin xyz="0 0 0.5" rpy="0 0 0"/> -->
-			<mass value="1"/>
-			<inertia ixx="2.3" ixy="0" ixz="0" iyy="3.35" iyz="0.00" izz="1.22" />
-		</inertial>
 		<visual>
 		    <origin xyz="1.05 0 0" rpy="0 0 0"/>
@@ -52,10 +75,7 @@
 			</geometry>
 		</collision>
+		<xacro:box_inertia m="35.0" w="3." d="2." h="1"/>
   	</link>
 	<link name="back_left_wheel">
-		<inertial>
-			<mass value="100"/>
-			<inertia ixx="0.2" ixy="0" ixz="0" iyy="0.2" iyz="0" izz="0.2"/>
-		</inertial>
   		<visual>
 		    <origin xyz="0 0 0" rpy="0 0 0"/>
@@ -73,10 +93,7 @@
 			</geometry>
 		</collision>
+		<xacro:cylinder_inertia m="55.5" r="0.5" h="0.2"/>
   	</link>
 	<link name="back_right_wheel">
-		<inertial>
-			<mass value="100"/>
-			<inertia ixx="0.2" ixy="0" ixz="0" iyy="0.2" iyz="0" izz="0.2"/>
-		</inertial>
   		<visual>
 		    <origin xyz="0 0 0" rpy="0 0 0"/>
@@ -94,10 +111,7 @@
 			</geometry>
 		</collision>
+		<xacro:cylinder_inertia m="55.5" r="0.5" h="0.2"/>
   	</link>
 	<link name="front_left_wheel">
-		<inertial>
-			<mass value="100"/>
-			<inertia ixx="0.2" ixy="0" ixz="0" iyy="0.2" iyz="0" izz="0.2"/>
-		</inertial>
   		<visual>
 		    <origin xyz="0 0 0" rpy="0 0 0"/>
@@ -115,10 +129,7 @@
 			</geometry>
 		</collision>
+		<xacro:cylinder_inertia m="55.5" r="0.5" h="0.2"/>
   	</link>
 	<link name="front_right_wheel">
-		<inertial>
-			<mass value="100"/>
-			<inertia ixx="0.2" ixy="0" ixz="0" iyy="0.2" iyz="0" izz="0.2"/>
-		</inertial>
   		<visual>
 		    <origin xyz="0 0 0" rpy="0 0 0"/>
@@ -136,11 +147,7 @@
 			</geometry>
 		</collision>
+		<xacro:cylinder_inertia m="55.5" r="0.5" h="0.2"/>
   	</link>
 	<link name="front_panel">
-		<inertial>
-			<origin xyz="0 1.95 0" rpy="0 0 0"/>
-			<mass value="100"/>
-			<inertia ixx="0.2" ixy="0" ixz="0" iyy="0.2" iyz="0" izz="0.2"/>
-		</inertial>
   		<visual>
 		    <origin xyz="0 1.95 0" rpy="0 0 0"/>
@@ -158,4 +165,5 @@
 			</geometry>
 		</collision>
+		<xacro:box_inertia m="10.0" w="4" d="5" h="6"/>
   	</link>
 	<link name="mid_panel">
@@ -175,4 +183,5 @@
 			</geometry>
 		</collision>
+		<xacro:box_inertia m="10.0" w="4" d="5" h="6"/>
   	</link>
 	<link name="mid_panel_prism">
@@ -186,5 +195,27 @@
 	     	</material>
 		</visual>
-  	</link>
+		<xacro:box_inertia m="10.0" w="4" d="5" h="6"/>
+  	</link>
+	<gazebo reference="base_link">
+		<material>Gazebo/Red</material>
+	</gazebo>
+	<gazebo reference="front_right_wheel">
+		<material>Gazebo/Green</material>
+	</gazebo>
+	<gazebo reference="front_left_wheel">
+		<material>Gazebo/Green</material>
+	</gazebo>
+	<gazebo reference="back_right_wheel">
+		<material>Gazebo/Green</material>
+	</gazebo>
+	<gazebo reference="back_left_wheel">
+		<material>Gazebo/Green</material>
+	</gazebo>
+	<gazebo reference="mid_panel">
+		<material>Gazebo/Green</material>
+	</gazebo>
+	<gazebo reference="front_panel">
+		<material>Gazebo/Red</material>
+	</gazebo>
 	<joint name="front_right_joint" type="continuous">
 		<origin xyz="-1.24 1.45 -0.07" rpy="0 1.57 0"/>

Commit message: Correction bugs

File: totem/bot/urdf/bot.urdf.xacro (robot description, xacro)
@@ -201,17 +201,17 @@
 	</gazebo>
 	<gazebo reference="front_right_wheel">
-		<material>Gazebo/Green</material>
+		<material>Gazebo/Blue</material>
 	</gazebo>
 	<gazebo reference="front_left_wheel">
-		<material>Gazebo/Green</material>
+		<material>Gazebo/Blue</material>
 	</gazebo>
 	<gazebo reference="back_right_wheel">
-		<material>Gazebo/Green</material>
+		<material>Gazebo/Blue</material>
 	</gazebo>
 	<gazebo reference="back_left_wheel">
-		<material>Gazebo/Green</material>
+		<material>Gazebo/Blue</material>
 	</gazebo>
 	<gazebo reference="mid_panel">
-		<material>Gazebo/Green</material>
+		<material>Gazebo/Blue</material>
 	</gazebo>
 	<gazebo reference="front_panel">
