Commit message: test

File: totem/bot/urdf/bot.urdf.xacro (robot description, xacro)
@@ -1,4 +1,10 @@
 <?xml version="1.0"?>
 <robot name="bot" xmlns:xacro="http://ros.org/wiki/xacro">
+	<xacro:property name="body_l" value="1" />
+	<xacro:property name="body_L" value="0.5" />
+	<xacro:property name="body_h" value="0.5" />
+	<xacro:property name="e" value="0.05" />
+	<xacro:property name="body_mass" value="30" />
+	<xacro:property name="wheel_mass" value="55.5" />
 	<!-- Define intertial property macros  -->
 	<xacro:macro name="box_inertia" params="m w h d">
@@ -22,179 +28,197 @@
 		</inertial>
 	</xacro:macro>
-	<link name="base_footprint"/>
-	<!-- The base footprint of the robot is located underneath the chassis -->
-	<joint name="base_joint" type="fixed">
-		<parent link="base_link"/>
-		<child link="base_footprint" />
-		<origin xyz="0.0 0.0 -0.1" rpy="0 0 0"/>
-	</joint>
- 	<link name="base_link">
+	<xacro:macro name="create_link" params="name mass *shape *inertia">
+		<link name="${name}">
+			<visual>
+				<geometry>
+					<xacro:insert_block name="shape" />
+				</geometry>
+			</visual>
+			<collision>
+				<geometry>
+					<xacro:insert_block name="shape" />
+				</geometry>
+			</collision>
+			<xacro:insert_block name="inertia" />
+		</link>
+	</xacro:macro>
+	<xacro:macro name="create_wheel" params="name mass *shape *inertia">
+		<xacro:create_link name="${name}" mass="${mass}">
+			<xacro:insert_block name="shape" />
+			<xacro:insert_block name="inertia" />
+ 	 	</xacro:create_link>
+		<gazebo reference="${name}">
+		<mu1>1.2</mu1>
+		<mu2>1.2</mu2>
+		<material>Gazebo/FlatBlack</material>
+		<kp>500000.0</kp>
+		<kd>10.0</kd>
+		<minDepth>0.001</minDepth>
+		<maxVel>0.1</maxVel>
+		</gazebo>
+	</xacro:macro>
+	<xacro:macro name="create_body" params="name mass">
+		<link name="${name}">
+			<visual>
+				<origin xyz="${(body_L/2)-e} 0 0" rpy="0 0 0"/>
+				<geometry>
+					<box size="${e} ${body_l} ${body_h}"/>
+				</geometry>
+				<material name="c">
+					<color rgba="0 0.9 0.9 1.0"/>
+				</material>
+			</visual>
+			<visual>
+				<origin xyz="${-(body_L/2)+e} 0 0" rpy="0 0 0"/>
+				<geometry>
+					<box size="${e} ${body_l} ${body_h}"/>
+				</geometry>
+				<material name="c">
+					<color rgba="0 0.9 0.9 1.0"/>
+				</material>
+			</visual>
+			<visual>
+				<origin xyz="0 ${(body_l/2)-e} 0" rpy="0 0 0"/>
+				<geometry>
+					<box size="${body_L} ${e} ${body_h}"/>
+				</geometry>
+				<material name="c">
+					<color rgba="0 0.9 0.9 1.0"/>
+				</material>
+			</visual>
+			<collision>
+				<origin xyz="${(body_L/2)-e} 0 0" rpy="0 0 0"/>
+				<geometry>
+					<box size="${e} ${body_l} ${body_h}"/>
+				</geometry>
+			</collision>
+			<collision>
+				<origin xyz="${-(body_L/2)+e} 0 0" rpy="0 0 0"/>
+				<geometry>
+					<box size="${e} ${body_l} ${body_h}"/>
+				</geometry>
+			</collision>
+			<collision>
+				<origin xyz="0 ${(body_L/2)-e} 0" rpy="0 0 0"/>
+				<geometry>
+					<box size="${body_L} ${e} ${body_h}"/>
+				</geometry>
+			</collision>
+			<xacro:box_inertia m="${mass}" w="3." d="2." h="1"/>
+		</link>
+	</xacro:macro>
+	<xacro:create_body name="base_link" mass="${body_mass}"/>
+	<!-- <link name="base_link">
 		<visual>
-		    <origin xyz="1.05 0 0" rpy="0 0 0"/>
-			<geometry>
-				<box size="0.1 4 1"/>
+			<origin xyz="${(body_L/2)-e} 0 0" rpy="0 0 0"/>
+			<geometry>
+				<box size="${e} ${body_l} ${body_h}"/>
 			</geometry>
 			<material name="c">
-	       		<color rgba="0 0.9 0.9 1.0"/>
-	     	</material>
+				<color rgba="0 0.9 0.9 1.0"/>
+			</material>
 		</visual>
-  		<visual>
-		    <origin xyz="-1.05 0 0" rpy="0 0 0"/>
-			<geometry>
-				<box size="0.1 4 1"/>
+		<visual>
+			<origin xyz="${-(body_L/2)+e} 0 0" rpy="0 0 0"/>
+			<geometry>
+				<box size="${e} ${body_l} ${body_h}"/>
 			</geometry>
 			<material name="c">
-	       		<color rgba="0 0.9 0.9 1.0"/>
-	     	</material>
+				<color rgba="0 0.9 0.9 1.0"/>
+			</material>
 		</visual>
-  		<visual>
-		    <origin xyz="0 -1.95 0" rpy="0 0 0"/>
-			<geometry>
-				<box size="2 0.1 1"/>
+		<visual>
+			<origin xyz="0 ${(body_l/2)-e} 0" rpy="0 0 0"/>
+			<geometry>
+				<box size="${body_L} ${e} ${body_h}"/>
 			</geometry>
 			<material name="c">
-	       		<color rgba="0 0.9 0.9 1.0"/>
-	     	</material>
+				<color rgba="0 0.9 0.9 1.0"/>
+			</material>
 		</visual>
 		<collision>
-		    <origin xyz="0 -1.95 0" rpy="0 0 0"/>
-			<geometry>
-				<box size="2 0.1 1"/>
+			<origin xyz="${(body_L/2)-e} 0 0" rpy="0 0 0"/>
+			<geometry>
+				<box size="${e} ${body_l} ${body_h}"/>
 			</geometry>
 		</collision>
 		<collision>
-		    <origin xyz="1.05 0 0" rpy="0 0 0"/>
-			<geometry>
-				<box size="0.1 4 1"/>
+			<origin xyz="${-(body_L/2)+e} 0 0" rpy="0 0 0"/>
+			<geometry>
+				<box size="${e} ${body_l} ${body_h}"/>
 			</geometry>
 		</collision>
 		<collision>
-		    <origin xyz="-1.05 0 0" rpy="0 0 0"/>
-			<geometry>
-				<box size="0.1 4 1"/>
+			<origin xyz="0 ${(body_L/2)-e} 0" rpy="0 0 0"/>
+			<geometry>
+				<box size="${body_L} ${e} ${body_h}"/>
 			</geometry>
 		</collision>
 		<xacro:box_inertia m="35.0" w="3." d="2." h="1"/>
-  	</link>
-	<link name="back_left_wheel">
-  		<visual>
-		    <origin xyz="0 0 0" rpy="0 0 0"/>
-			<geometry>
-				<cylinder radius="0.5" length="0.2"/>
-			</geometry>
-			<material name="d">
-	       		<color rgba="0 0 0 0"/>
-	     	</material>
+	</link> -->
+	<xacro:create_wheel name="back_left_wheel" mass="${wheel_mass}">
+		<cylinder length="${body_h/2}" radius="0.1"/>
+		<xacro:cylinder_inertia m="${wheel_mass}" r="${body_h/2}" h="0.1" />
+	</xacro:create_wheel>
+	<xacro:create_wheel name="back_right_wheel" mass="${wheel_mass}">
+		<cylinder length="${body_h/2}" radius="0.1"/>
+		<xacro:cylinder_inertia m="${wheel_mass}" r="${body_h/2}" h="0.1" />
+	</xacro:create_wheel>
+	<xacro:create_wheel name="front_left_wheel" mass="${wheel_mass}">
+		<cylinder length="${body_h/2}" radius="0.1"/>
+		<xacro:cylinder_inertia m="${wheel_mass}" r="${body_h/2}" h="0.1" />
+	</xacro:create_wheel>
+	<xacro:create_wheel name="front__wheel" mass="${wheel_mass}">
+		<cylinder length="${body_h/2}" radius="0.1"/>
+		<xacro:cylinder_inertia m="${wheel_mass}" r="${body_h/2}" h="0.1" />
+	</xacro:create_wheel>
+	<!-- <link name="front_panel">
+		<visual>
+			<origin xyz="0 ${(body_l/2)-e} 0" rpy="0 0 0"/>
+			<geometry>
+				<box size="${body_L} ${e} ${body_h}"/>
+			</geometry>
+			<material name="f">
+				<color rgba="0 0 0.9 1.0"/>
+			</material>
 		</visual>
 		<collision>
-		    <origin xyz="0 0 0" rpy="0 0 0"/>
-			<geometry>
-				<cylinder radius="0.5" length="0.2"/>
-			</geometry>
-		</collision>
-		<xacro:cylinder_inertia m="55.5" r="0.5" h="0.2"/>
-  	</link>
-	<link name="back_right_wheel">
-  		<visual>
-		    <origin xyz="0 0 0" rpy="0 0 0"/>
-			<geometry>
-				<cylinder radius="0.5" length="0.2"/>
-			</geometry>
-			<material name="d">
-	       		<color rgba="0 0 0 0"/>
-	     	</material>
-		</visual>
-		<collision>
-		    <origin xyz="0 0 0" rpy="0 0 0"/>
-			<geometry>
-				<cylinder radius="0.5" length="0.2"/>
-			</geometry>
-		</collision>
-		<xacro:cylinder_inertia m="55.5" r="0.5" h="0.2"/>
-  	</link>
-	<link name="front_left_wheel">
-  		<visual>
-		    <origin xyz="0 0 0" rpy="0 0 0"/>
-			<geometry>
-				<cylinder radius="0.5" length="0.2"/>
-			</geometry>
-			<material name="d">
-	       		<color rgba="0 0 0 0"/>
-	     	</material>
-		</visual>
-		<collision>
-		    <origin xyz="0 0 0" rpy="0 0 0"/>
-			<geometry>
-				<cylinder radius="0.5" length="0.2"/>
-			</geometry>
-		</collision>
-		<xacro:cylinder_inertia m="55.5" r="0.5" h="0.2"/>
-  	</link>
-	<link name="front_right_wheel">
-  		<visual>
-		    <origin xyz="0 0 0" rpy="0 0 0"/>
-			<geometry>
-				<cylinder radius="0.5" length="0.2"/>
-			</geometry>
-			<material name="d">
-	       		<color rgba="0 0 0 0"/>
-	     	</material>
-		</visual>
-		<collision>
-		    <origin xyz="0 0 0" rpy="0 0 0"/>
-			<geometry>
-				<cylinder radius="0.5" length="0.2"/>
-			</geometry>
-		</collision>
-		<xacro:cylinder_inertia m="55.5" r="0.5" h="0.2"/>
-  	</link>
-	<link name="front_panel">
-  		<visual>
-		    <origin xyz="0 1.95 0" rpy="0 0 0"/>
-			<geometry>
-				<box size="2 0.1 1"/>
-			</geometry>
-			<material name="f">
-	       		<color rgba="0 0 0.9 1.0"/>
-	     	</material>
-		</visual>
-		<collision>
-		    <origin xyz="0 1.95 0" rpy="0 0 0"/>
-			<geometry>
-				<box size="2 0.1 1"/>
+			<origin xyz="0 ${(body_l/2)-e} 0" rpy="0 0 0"/>
+			<geometry>
+				<box size="${body_L} ${e} ${body_h}"/>
 			</geometry>
 		</collision>
 		<xacro:box_inertia m="10.0" w="4" d="5" h="6"/>
-  	</link>
+	</link>
 	<link name="mid_panel">
-  		<visual>
-		    <origin xyz="0 0 0" rpy="0 0 0"/>
-			<geometry>
-				<box size="1.9 0.02 1"/>
-			</geometry>
-			<material name="l">
-	       		<color rgba="1 0 0 1.0"/>
-	     	</material>
-		</visual>
-		<collision>
-		    <origin xyz="0 0 0" rpy="0 0 0"/>
-			<geometry>
-				<box size="1.9 0.02 1"/>
-			</geometry>
-		</collision>
-		<xacro:box_inertia m="10.0" w="4" d="5" h="6"/>
-  	</link>
+			<visual>
+				<origin xyz="0 0 0" rpy="0 0 0"/>
+				<geometry>
+					<box size="${body_L-0.2} 0.02 ${body_h}"/>
+				</geometry>
+				<material name="l">
+					<color rgba="1 0 0 1.0"/>
+				</material>
+			</visual>
+			<collision>
+				<origin xyz="0 0 0" rpy="0 0 0"/>
+				<geometry>
+					<box size="${body_L-0.2} 0.02 ${body_h}"/>
+				</geometry>
+			</collision>
+			<xacro:box_inertia m="10.0" w="4" d="5" h="6"/>
+	</link>
 	<link name="mid_panel_prism">
-  		<visual>
-		    <origin xyz="-0.975 0 0" rpy="0 0 0"/>
-			<geometry>
-				<box size="0.05 0.1 0.1"/>
-			</geometry>
-			<material name="m">
-	       		<color rgba="1 1 0 1.0"/>
-	     	</material>
-		</visual>
-		<xacro:box_inertia m="10.0" w="4" d="5" h="6"/>
-  	</link>
+			<visual>
+				<origin xyz="-0.975 0 0" rpy="0 0 0"/>
+				<geometry>
+					<box size="0.05 0.1 0.1"/>
+				</geometry>
+				<material name="m">
+					<color rgba="1 1 0 1.0"/>
+				</material>
+			</visual>
+			<xacro:box_inertia m="10.0" w="4" d="5" h="6"/>
+	</link> -->
 	<gazebo reference="base_link">
 		<material>Gazebo/Red</material>
@@ -219,69 +243,70 @@
 	</gazebo>
 	<joint name="front_right_joint" type="continuous">
-		<origin xyz="-1.24 1.45 -0.07" rpy="0 1.57 0"/>
-        <parent link="base_link"/>
-        <child link="front_right_wheel"/>
+		<origin xyz="${-((body_l/2) + e + 0.2)} ${(body_l/2)-(body_h/2)-0.05} -0.07" rpy="0 1.57 0"/>
+		<parent link="base_link"/>
+		<child link="front_right_wheel"/>
 		<limit effort="30" velocity="2.0"/>
-      	<axis xyz="0 0 1" />
-      	<dynamics damping="1.0" />
- 	</joint>
+		<axis xyz="0 0 1" />
+		<dynamics damping="1.0" />
+	</joint>
 	<joint name="front_left_joint" type="continuous">
-		<origin xyz="1.24 1.45 -0.07" rpy="0 1.57 0"/>
-        <parent link="base_link"/>
-        <child link="front_left_wheel"/>
+		<origin xyz="${(body_l/2) + e + 0.2} ${(body_l/2)-(body_h/2)-0.05} -0.07" rpy="0 1.57 0"/>
+		<parent link="base_link"/>
+		<child link="front_left_wheel"/>
 		<axis xyz="0 0 1"/>
 		<limit effort="30" velocity="2.0"/>
- 	</joint>
+	</joint>
 	<joint name="back_right_joint" type="continuous">
-		<origin xyz="-1.24 -1.45 -0.07" rpy="0 1.57 0"/>
-        <parent link="base_link"/>
-        <child link="back_right_wheel"/>
+		<origin xyz="${-((body_l/2) + e + 0.2)} ${-(body_l/2)-(body_h/2)-0.05} -0.07" rpy="0 1.57 0"/>
+		<parent link="base_link"/>
+		<child link="back_right_wheel"/>
 		<axis xyz="0 0 1"/>
 		<limit effort="30" velocity="2.0"/>
- 	</joint>
+	</joint>
 	<joint name="back_left_joint" type="continuous">
-		<origin xyz="1.24 -1.45 -0.07" rpy="0 1.57 0"/>
-        <parent link="base_link"/>
-        <child link="back_left_wheel"/>
+		<origin xyz="${(body_l/2) + e + 0.2} ${-(body_l/2)-(body_h/2)-0.05} -0.07" rpy="0 1.57 0"/>
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
Commit message: parametrer le fichier urdf

File: totem/bot/urdf/bot.urdf.xacro (robot description, xacro)
@@ -58,56 +58,53 @@
 		</gazebo>
 	</xacro:macro>
-	<xacro:macro name="create_body" params="name mass">
-		<link name="${name}">
-			<visual>
-				<origin xyz="${(body_L/2)-e} 0 0" rpy="0 0 0"/>
-				<geometry>
-					<box size="${e} ${body_l} ${body_h}"/>
-				</geometry>
-				<material name="c">
-					<color rgba="0 0.9 0.9 1.0"/>
-				</material>
-			</visual>
-			<visual>
-				<origin xyz="${-(body_L/2)+e} 0 0" rpy="0 0 0"/>
-				<geometry>
-					<box size="${e} ${body_l} ${body_h}"/>
-				</geometry>
-				<material name="c">
-					<color rgba="0 0.9 0.9 1.0"/>
-				</material>
-			</visual>
-			<visual>
-				<origin xyz="0 ${(body_l/2)-e} 0" rpy="0 0 0"/>
-				<geometry>
-					<box size="${body_L} ${e} ${body_h}"/>
-				</geometry>
-				<material name="c">
-					<color rgba="0 0.9 0.9 1.0"/>
-				</material>
-			</visual>
-			<collision>
-				<origin xyz="${(body_L/2)-e} 0 0" rpy="0 0 0"/>
-				<geometry>
-					<box size="${e} ${body_l} ${body_h}"/>
-				</geometry>
-			</collision>
-			<collision>
-				<origin xyz="${-(body_L/2)+e} 0 0" rpy="0 0 0"/>
-				<geometry>
-					<box size="${e} ${body_l} ${body_h}"/>
-				</geometry>
-			</collision>
-			<collision>
-				<origin xyz="0 ${(body_L/2)-e} 0" rpy="0 0 0"/>
-				<geometry>
-					<box size="${body_L} ${e} ${body_h}"/>
-				</geometry>
-			</collision>
-			<xacro:box_inertia m="${mass}" w="3." d="2." h="1"/>
-		</link>
-	</xacro:macro>
-	<xacro:create_body name="base_link" mass="${body_mass}"/>
-	<!-- <link name="base_link">
+	<link name="base_link">
+		<visual>
+			<origin xyz="${(body_L/2)-e} 0 0" rpy="0 0 0"/>
+			<geometry>
+				<box size="${e} ${body_l} ${body_h}"/>
+			</geometry>
+			<material name="c">
+				<color rgba="0 0.9 0.9 1.0"/>
+			</material>
+		</visual>
+		<visual>
+			<origin xyz="${-(body_L/2)+e} 0 0" rpy="0 0 0"/>
+			<geometry>
+				<box size="${e} ${body_l} ${body_h}"/>
+			</geometry>
+			<material name="c">
+				<color rgba="0 0.9 0.9 1.0"/>
+			</material>
+		</visual>
+		<visual>
+			<origin xyz="0 ${(body_l/2)-e} 0" rpy="0 0 0"/>
+			<geometry>
+				<box size="${body_L} ${e} ${body_h}"/>
+			</geometry>
+			<material name="c">
+				<color rgba="0 0.9 0.9 1.0"/>
+			</material>
+		</visual>
+		<collision>
+			<origin xyz="${(body_L/2)-e} 0 0" rpy="0 0 0"/>
+			<geometry>
+				<box size="${e} ${body_l} ${body_h}"/>
+			</geometry>
+		</collision>
+		<collision>
+			<origin xyz="${-(body_L/2)+e} 0 0" rpy="0 0 0"/>
+			<geometry>
+				<box size="${e} ${body_l} ${body_h}"/>
+			</geometry>
+		</collision>
+		<collision>
+			<origin xyz="0 ${(body_L/2)-e} 0" rpy="0 0 0"/>
+			<geometry>
+				<box size="${body_L} ${e} ${body_h}"/>
+			</geometry>
+		</collision>
+		<xacro:box_inertia m="${mass}" w="3." d="2." h="1"/>
+	</link>
+	<link name="base_link">
 		<visual>
 			<origin xyz="${(body_L/2)-e} 0 0" rpy="0 0 0"/>
@@ -210,14 +207,14 @@
 	</link>
 	<link name="mid_panel_prism">
-			<visual>
-				<origin xyz="-0.975 0 0" rpy="0 0 0"/>
-				<geometry>
-					<box size="0.05 0.1 0.1"/>
-				</geometry>
-				<material name="m">
-					<color rgba="1 1 0 1.0"/>
-				</material>
-			</visual>
-			<xacro:box_inertia m="10.0" w="4" d="5" h="6"/>
+		<visual>
+			<origin xyz="-0.975 0 0" rpy="0 0 0"/>
+			<geometry>
+				<box size="0.05 0.1 0.1"/>
+			</geometry>
+			<material name="m">
+				<color rgba="1 1 0 1.0"/>
+			</material>
+		</visual>
+		<xacro:box_inertia m="10.0" w="4" d="5" h="6"/>
 	</link> -->
 	<gazebo reference="base_link">
