Commit message: change robot size

File: totem/bot/urdf/bot.urdf.xacro (robot description, xacro)
@@ -1,10 +1,4 @@
 <?xml version="1.0"?>
 <robot name="bot" xmlns:xacro="http://ros.org/wiki/xacro">
-	<xacro:property name="body_l" value="1" />
-	<xacro:property name="body_L" value="0.5" />
-	<xacro:property name="body_h" value="0.5" />
-	<xacro:property name="e" value="0.05" />
-	<xacro:property name="body_mass" value="30" />
-	<xacro:property name="wheel_mass" value="55.5" />
 	<!-- Define intertial property macros  -->
 	<xacro:macro name="box_inertia" params="m w h d">
@@ -28,211 +22,196 @@
 		</inertial>
 	</xacro:macro>
-	<xacro:macro name="create_link" params="name mass *shape *inertia">
-		<link name="${name}">
-			<visual>
-				<geometry>
-					<xacro:insert_block name="shape" />
-				</geometry>
-			</visual>
-			<collision>
-				<geometry>
-					<xacro:insert_block name="shape" />
-				</geometry>
-			</collision>
-			<xacro:insert_block name="inertia" />
-		</link>
-	</xacro:macro>
-	<xacro:macro name="create_wheel" params="name mass *shape *inertia">
-		<xacro:create_link name="${name}" mass="${mass}">
-			<xacro:insert_block name="shape" />
-			<xacro:insert_block name="inertia" />
- 	 	</xacro:create_link>
-		<gazebo reference="${name}">
-		<mu1>1.2</mu1>
-		<mu2>1.2</mu2>
-		<material>Gazebo/FlatBlack</material>
-		<kp>500000.0</kp>
-		<kd>10.0</kd>
-		<minDepth>0.001</minDepth>
-		<maxVel>0.1</maxVel>
-		</gazebo>
-	</xacro:macro>
-	<link name="base_link">
+	<link name="base_footprint"/>
+	<!-- The base footprint of the robot is located underneath the chassis -->
+	<joint name="base_joint" type="fixed">
+		<parent link="base_link"/>
+		<child link="base_footprint" />
+		<origin xyz="0.0 0.0 -0.1" rpy="0 0 0"/>
+	</joint>
+ 	<link name="base_link">
 		<visual>
-			<origin xyz="${(body_L/2)-e} 0 0" rpy="0 0 0"/>
-			<geometry>
-				<box size="${e} ${body_l} ${body_h}"/>
+		    <origin xyz="0.4 0 0" rpy="0 0 0"/>
+			<geometry>
+				<box size="0.1 1.5 0.5"/>
 			</geometry>
 			<material name="c">
-				<color rgba="0 0.9 0.9 1.0"/>
-			</material>
-		</visual>
-		<visual>
-			<origin xyz="${-(body_L/2)+e} 0 0" rpy="0 0 0"/>
-			<geometry>
-				<box size="${e} ${body_l} ${body_h}"/>
+	       		<color rgba="0 0.9 0.9 1.0"/>
+	     	</material>
+		</visual>
+  		<visual>
+		    <origin xyz="-0.4 0 0" rpy="0 0 0"/>
+			<geometry>
+				<box size="0.1 1.5 0.5"/>
 			</geometry>
 			<material name="c">
-				<color rgba="0 0.9 0.9 1.0"/>
-			</material>
-		</visual>
-		<visual>
-			<origin xyz="0 ${(body_l/2)-e} 0" rpy="0 0 0"/>
-			<geometry>
-				<box size="${body_L} ${e} ${body_h}"/>
+	       		<color rgba="0 0.9 0.9 1.0"/>
+	     	</material>
+		</visual>
+  		<visual>
+		    <origin xyz="0 -0.7 0" rpy="0 0 0"/>
+			<geometry>
+				<box size="0.7 0.1 0.5"/>
 			</geometry>
 			<material name="c">
-				<color rgba="0 0.9 0.9 1.0"/>
-			</material>
-		</visual>
-		<collision>
-			<origin xyz="${(body_L/2)-e} 0 0" rpy="0 0 0"/>
-			<geometry>
-				<box size="${e} ${body_l} ${body_h}"/>
-			</geometry>
-		</collision>
-		<collision>
-			<origin xyz="${-(body_L/2)+e} 0 0" rpy="0 0 0"/>
-			<geometry>
-				<box size="${e} ${body_l} ${body_h}"/>
-			</geometry>
-		</collision>
-		<collision>
-			<origin xyz="0 ${(body_L/2)-e} 0" rpy="0 0 0"/>
-			<geometry>
-				<box size="${body_L} ${e} ${body_h}"/>
-			</geometry>
-		</collision>
-		<xacro:box_inertia m="${mass}" w="3." d="2." h="1"/>
-	</link>
-	<link name="base_link">
-		<visual>
-			<origin xyz="${(body_L/2)-e} 0 0" rpy="0 0 0"/>
-			<geometry>
-				<box size="${e} ${body_l} ${body_h}"/>
-			</geometry>
-			<material name="c">
-				<color rgba="0 0.9 0.9 1.0"/>
-			</material>
-		</visual>
-		<visual>
-			<origin xyz="${-(body_L/2)+e} 0 0" rpy="0 0 0"/>
-			<geometry>
-				<box size="${e} ${body_l} ${body_h}"/>
-			</geometry>
-			<material name="c">
-				<color rgba="0 0.9 0.9 1.0"/>
-			</material>
-		</visual>
-		<visual>
-			<origin xyz="0 ${(body_l/2)-e} 0" rpy="0 0 0"/>
-			<geometry>
-				<box size="${body_L} ${e} ${body_h}"/>
-			</geometry>
-			<material name="c">
-				<color rgba="0 0.9 0.9 1.0"/>
-			</material>
-		</visual>
-		<collision>
-			<origin xyz="${(body_L/2)-e} 0 0" rpy="0 0 0"/>
-			<geometry>
-				<box size="${e} ${body_l} ${body_h}"/>
-			</geometry>
-		</collision>
-		<collision>
-			<origin xyz="${-(body_L/2)+e} 0 0" rpy="0 0 0"/>
-			<geometry>
-				<box size="${e} ${body_l} ${body_h}"/>
-			</geometry>
-		</collision>
-		<collision>
-			<origin xyz="0 ${(body_L/2)-e} 0" rpy="0 0 0"/>
-			<geometry>
-				<box size="${body_L} ${e} ${body_h}"/>
+	       		<color rgba="0 0.9 0.9 1.0"/>
+	     	</material>
+		</visual>
+		<collision>
+		    <origin xyz="0 -0.7 0" rpy="0 0 0"/>
+			<geometry>
+				<box size="0.7 0.1 0.5"/>
+			</geometry>
+		</collision>
+		<collision>
+		    <origin xyz="0.4  0 0" rpy="0 0 0"/>
+			<geometry>
+				<box size="0.1 1.5 0.5"/>
+			</geometry>
+		</collision>
+		<collision>
+		    <origin xyz="-0.4 0 0" rpy="0 0 0"/>
+			<geometry>
+				<box size="0.1 1.5 0.5"/>
 			</geometry>
 		</collision>
 		<xacro:box_inertia m="35.0" w="3." d="2." h="1"/>
-	</link> -->
-	<xacro:create_wheel name="back_left_wheel" mass="${wheel_mass}">
-		<cylinder length="${body_h/2}" radius="0.1"/>
-		<xacro:cylinder_inertia m="${wheel_mass}" r="${body_h/2}" h="0.1" />
-	</xacro:create_wheel>
-	<xacro:create_wheel name="back_right_wheel" mass="${wheel_mass}">
-		<cylinder length="${body_h/2}" radius="0.1"/>
-		<xacro:cylinder_inertia m="${wheel_mass}" r="${body_h/2}" h="0.1" />
-	</xacro:create_wheel>
-	<xacro:create_wheel name="front_left_wheel" mass="${wheel_mass}">
-		<cylinder length="${body_h/2}" radius="0.1"/>
-		<xacro:cylinder_inertia m="${wheel_mass}" r="${body_h/2}" h="0.1" />
-	</xacro:create_wheel>
-	<xacro:create_wheel name="front__wheel" mass="${wheel_mass}">
-		<cylinder length="${body_h/2}" radius="0.1"/>
-		<xacro:cylinder_inertia m="${wheel_mass}" r="${body_h/2}" h="0.1" />
-	</xacro:create_wheel>
-	<!-- <link name="front_panel">
-		<visual>
-			<origin xyz="0 ${(body_l/2)-e} 0" rpy="0 0 0"/>
-			<geometry>
-				<box size="${body_L} ${e} ${body_h}"/>
+  	</link>
+	<link name="back_left_wheel">
+  		<visual>
+		    <origin xyz="0 0 0" rpy="0 0 0"/>
+			<geometry>
+				<cylinder radius="0.25" length="0.1"/>
+			</geometry>
+			<material name="d">
+	       		<color rgba="0 0 0 0"/>
+	     	</material>
+		</visual>
+		<collision>
+		    <origin xyz="0 0 0" rpy="0 0 0"/>
+			<geometry>
+				<cylinder radius="0.25" length="0.1"/>
+			</geometry>
+		</collision>
+		<xacro:cylinder_inertia m="2" r="0.25" h="0.2"/>
+  	</link>
+	<link name="back_right_wheel">
+  		<visual>
+		    <origin xyz="0 0 0" rpy="0 0 0"/>
+			<geometry>
+				<cylinder radius="0.25" length="0.1"/>
+			</geometry>
+			<material name="d">
+	       		<color rgba="0 0 0 0"/>
+	     	</material>
+		</visual>
+		<collision>
+		    <origin xyz="0 0 0" rpy="0 0 0"/>
+			<geometry>
+				<cylinder radius="0.25" length="0.1"/>
+			</geometry>
+		</collision>
+		<xacro:cylinder_inertia m="2" r="0.25" h="0.1"/>
+  	</link>
+	<link name="front_left_wheel">
+  		<visual>
+		    <origin xyz="0 0 0" rpy="0 0 0"/>
+			<geometry>
+				<cylinder radius="0.25" length="0.1"/>
+			</geometry>
+			<material name="d">
+	       		<color rgba="0 0 0 0"/>
+	     	</material>
+		</visual>
+		<collision>
+		    <origin xyz="0 0 0" rpy="0 0 0"/>
+			<geometry>
+				<cylinder radius="0.25" length="0.1"/>
+			</geometry>
+		</collision>
+		<xacro:cylinder_inertia m="2" r="0.25" h="0.1"/>
+  	</link>
+	<link name="front_right_wheel">
+  		<visual>
+		    <origin xyz="0 0 0" rpy="0 0 0"/>
+			<geometry>
+				<cylinder radius="0.25" length="0.1"/>
+			</geometry>
+			<material name="d">
+	       		<color rgba="0 0 0 0"/>
+	     	</material>
+		</visual>
+		<collision>
+		    <origin xyz="0 0 0" rpy="0 0 0"/>
+			<geometry>
+				<cylinder radius="0.25" length="0.1"/>
+			</geometry>
+		</collision>
+		<xacro:cylinder_inertia m="2" r="0.25" h="0.1"/>
+  	</link>
+	<link name="front_panel">
+  		<visual>
+		    <origin xyz="0 0.7 0" rpy="0 0 0"/>
+			<geometry>
+				<box size="0.7 0.1 0.5"/>
 			</geometry>
 			<material name="f">
-				<color rgba="0 0 0.9 1.0"/>
-			</material>
-		</visual>
-		<collision>
-			<origin xyz="0 ${(body_l/2)-e} 0" rpy="0 0 0"/>
-			<geometry>
-				<box size="${body_L} ${e} ${body_h}"/>
-			</geometry>
-		</collision>
-		<xacro:box_inertia m="10.0" w="4" d="5" h="6"/>
-	</link>
+	       		<color rgba="0 0 0.9 1.0"/>
+	     	</material>
+		</visual>
+		<collision>
+		    <origin xyz="0 0.7 0" rpy="0 0 0"/>
+			<geometry>
+				<box size="0.7 0.1 0.5"/>
+			</geometry>
+		</collision>
+		<xacro:box_inertia m="10.0" w="0.7" d="0.1" h="0.5"/>
+  	</link>
 	<link name="mid_panel">
-			<visual>
-				<origin xyz="0 0 0" rpy="0 0 0"/>
-				<geometry>
-					<box size="${body_L-0.2} 0.02 ${body_h}"/>
-				</geometry>
-				<material name="l">
-					<color rgba="1 0 0 1.0"/>
-				</material>
-			</visual>
-			<collision>
-				<origin xyz="0 0 0" rpy="0 0 0"/>
-				<geometry>
-					<box size="${body_L-0.2} 0.02 ${body_h}"/>
-				</geometry>
-			</collision>
-			<xacro:box_inertia m="10.0" w="4" d="5" h="6"/>
-	</link>
+  		<visual>
+		    <origin xyz="0 0 0" rpy="0 0 0"/>
+			<geometry>
+				<box size="0.6 0.02 0.5"/>
+			</geometry>
+			<material name="l">
+	       		<color rgba="1 0 0 1.0"/>
+	     	</material>
+		</visual>
+		<collision>
+		    <origin xyz="0 0 0" rpy="0 0 0"/>
+			<geometry>
+				<box size="0.9 0.02 0.5"/>
+			</geometry>
+		</collision>
+		<xacro:box_inertia m="10.0" w="0.9" d="0.02" h="1"/>
+  	</link>
 	<link name="mid_panel_prism">
-		<visual>
-			<origin xyz="-0.975 0 0" rpy="0 0 0"/>
+  		<visual>
+		    <origin xyz="-0.335 0 0" rpy="0 0 0"/>
 			<geometry>
 				<box size="0.05 0.1 0.1"/>
 			</geometry>
 			<material name="m">
-				<color rgba="1 1 0 1.0"/>
-			</material>
-		</visual>
-		<xacro:box_inertia m="10.0" w="4" d="5" h="6"/>
-	</link> -->
+	       		<color rgba="1 1 0 1.0"/>
+	     	</material>
+		</visual>
+		<xacro:box_inertia m="0" w="0.05" d="0.1" h="0.1"/>
+  	</link>
 	<gazebo reference="base_link">
 		<material>Gazebo/Red</material>
 	</gazebo>
 	<gazebo reference="front_right_wheel">
-		<material>Gazebo/Green</material>
+		<material>Gazebo/Blue</material>
 	</gazebo>
 	<gazebo reference="front_left_wheel">
-		<material>Gazebo/Green</material>
+		<material>Gazebo/Blue</material>
 	</gazebo>
 	<gazebo reference="back_right_wheel">
-		<material>Gazebo/Green</material>
+		<material>Gazebo/Blue</material>
 	</gazebo>
 	<gazebo reference="back_left_wheel">
-		<material>Gazebo/Green</material>
+		<material>Gazebo/Blue</material>
 	</gazebo>
 	<gazebo reference="mid_panel">
-		<material>Gazebo/Green</material>
+		<material>Gazebo/Blue</material>
 	</gazebo>
 	<gazebo reference="front_panel">
@@ -240,70 +219,69 @@
 	</gazebo>
 	<joint name="front_right_joint" type="continuous">
-		<origin xyz="${-((body_l/2) + e + 0.2)} ${(body_l/2)-(body_h/2)-0.05} -0.07" rpy="0 1.57 0"/>
-		<parent link="base_link"/>
-		<child link="front_right_wheel"/>
+		<origin xyz="-0.51 0.5 -0.07" rpy="0 1.57 0"/>
+        <parent link="base_link"/>
+        <child link="front_right_wheel"/>
 		<limit effort="30" velocity="2.0"/>
-		<axis xyz="0 0 1" />
-		<dynamics damping="1.0" />
-	</joint>
+      	<axis xyz="0 0 1" />
+      	<dynamics damping="1.0" />
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
Commit message: Rob architecture change

File: totem/bot/urdf/bot.urdf.xacro (robot description, xacro)
@@ -35,43 +35,52 @@
 				<box size="0.1 1.5 0.5"/>
 			</geometry>
+			<material name="c1">
+	       		<color rgba="0 0.5 0.9 1.0"/>
+	     	</material>
+		</visual>
+  		<visual>
+		    <origin xyz="-0.4 0 0" rpy="0 0 0"/>
+			<geometry>
+				<box size="0.1 1.5 0.5"/>
+			</geometry>
 			<material name="c">
+	       		<color rgba="0 0.5 0.9 1.0"/>
+	     	</material>
+		</visual>
+  		<visual>
+		    <origin xyz="0 -0.7 0" rpy="0 0 0"/>
+			<geometry>
+				<box size="0.7 0.1 0.5"/>
+			</geometry>
+			<material name="c2">
 	       		<color rgba="0 0.9 0.9 1.0"/>
 	     	</material>
 		</visual>
   		<visual>
+          	<origin xyz="0 -0.2 0" rpy="0 0 0"/>
+			<geometry>
+				<box size="0.7 0.95 0.5"/>
+			</geometry>
+			<material name="c">
+	       		<color rgba="0 0.1 0.9 1.0"/>
+	     	</material>
+		</visual>
+		<collision>
+		    <origin xyz="0 -0.7 0" rpy="0 0 0"/>
+			<geometry>
+				<box size="0.7 0.1 0.5"/>
+			</geometry>
+		</collision>
+		<collision>
+		    <origin xyz="0.4  0 0" rpy="0 0 0"/>
+			<geometry>
+				<box size="0.1 1.5 0.5"/>
+			</geometry>
+		</collision>
+		<collision>
 		    <origin xyz="-0.4 0 0" rpy="0 0 0"/>
 			<geometry>
 				<box size="0.1 1.5 0.5"/>
 			</geometry>
-			<material name="c">
-	       		<color rgba="0 0.9 0.9 1.0"/>
-	     	</material>
-		</visual>
-  		<visual>
-		    <origin xyz="0 -0.7 0" rpy="0 0 0"/>
-			<geometry>
-				<box size="0.7 0.1 0.5"/>
-			</geometry>
-			<material name="c">
-	       		<color rgba="0 0.9 0.9 1.0"/>
-	     	</material>
-		</visual>
-		<collision>
-		    <origin xyz="0 -0.7 0" rpy="0 0 0"/>
-			<geometry>
-				<box size="0.7 0.1 0.5"/>
-			</geometry>
-		</collision>
-		<collision>
-		    <origin xyz="0.4  0 0" rpy="0 0 0"/>
-			<geometry>
-				<box size="0.1 1.5 0.5"/>
-			</geometry>
-		</collision>
-		<collision>
-		    <origin xyz="-0.4 0 0" rpy="0 0 0"/>
-			<geometry>
-				<box size="0.1 1.5 0.5"/>
-			</geometry>
 		</collision>
 		<xacro:box_inertia m="35.0" w="3." d="2." h="1"/>
@@ -113,5 +122,23 @@
 		<xacro:cylinder_inertia m="2" r="0.25" h="0.1"/>
   	</link>
-	<link name="front_left_wheel">
+	<link name="mid_wheel">
+  		<visual>
+		    <origin xyz="0 0 0" rpy="0 0 0"/>
+			<geometry>
+				<sphere radius="0.02"/>
+			</geometry>
+			<material name="d">
+	       		<color rgba="0 0 0 0"/>
+	     	</material>
+		</visual>
+		<collision>
+		    <origin xyz="0 0 0" rpy="0 0 0"/>
+			<geometry>
+				<sphere radius="0.02"/>
+			</geometry>
+		</collision>
+		<xacro:sphere_inertia m="1" r="0.02"/>
+  	</link>
+	<!-- <link name="front_left_wheel">
   		<visual>
 		    <origin xyz="0 0 0" rpy="0 0 0"/>
@@ -148,5 +175,5 @@
 		</collision>
 		<xacro:cylinder_inertia m="2" r="0.25" h="0.1"/>
-  	</link>
+  	</link> -->
 	<link name="front_panel">
   		<visual>
@@ -167,5 +194,14 @@
 		<xacro:box_inertia m="10.0" w="0.7" d="0.1" h="0.5"/>
   	</link>
-	<link name="mid_panel">
+	<gazebo reference="mid_wheel">
+		<mu1>0.01</mu1>
+		<mu2>0.01</mu2>
+		<material>Gazebo/SkyBlue</material>
+		<kp>500000.0</kp>
+		<kd>1.0</kd>
+		<minDepth>0.001</minDepth>
+		<maxVel>0.1</maxVel>
+	</gazebo>
+	<!-- <link name="mid_panel">
   		<visual>
 		    <origin xyz="0 0 0" rpy="0 0 0"/>
@@ -196,14 +232,14 @@
 		</visual>
 		<xacro:box_inertia m="0" w="0.05" d="0.1" h="0.1"/>
-  	</link>
+  	</link> -->
 	<gazebo reference="base_link">
 		<material>Gazebo/Red</material>
 	</gazebo>
-	<gazebo reference="front_right_wheel">
+	<!-- <gazebo reference="front_right_wheel">
 		<material>Gazebo/Blue</material>
 	</gazebo>
 	<gazebo reference="front_left_wheel">
 		<material>Gazebo/Blue</material>
-	</gazebo>
+	</gazebo> -->
 	<gazebo reference="back_right_wheel">
 		<material>Gazebo/Blue</material>
@@ -212,11 +248,11 @@
 		<material>Gazebo/Blue</material>
 	</gazebo>
-	<gazebo reference="mid_panel">
-		<material>Gazebo/Blue</material>
-	</gazebo>
+	<!-- <gazebo reference="mid_panel">
+		<material>Gazebo/Blue</material>
+	</gazebo> -->
 	<gazebo reference="front_panel">
 		<material>Gazebo/Red</material>
 	</gazebo>
-	<joint name="front_right_joint" type="continuous">
+	<!-- <joint name="front_right_joint" type="continuous">
 		<origin xyz="-0.51 0.5 -0.07" rpy="0 1.57 0"/>
         <parent link="base_link"/>
@@ -232,18 +268,23 @@
 		<axis xyz="0 0 1"/>
 		<limit effort="30" velocity="2.0"/>
- 	</joint>
+ 	</joint> -->
 	<joint name="back_right_joint" type="continuous">
-		<origin xyz="-0.51 -0.5 -0.07" rpy="0 1.57 0"/>
+		<origin xyz="-0.51 -0.5 -0.02" rpy="0 1.57 0"/>
         <parent link="base_link"/>
         <child link="back_right_wheel"/>
 		<axis xyz="0 0 1"/>
-		<limit effort="30" velocity="2.0"/>
+		<limit effort="30" velocity="10.0"/>
  	</joint>
 	<joint name="back_left_joint" type="continuous">
-		<origin xyz="0.51 -0.5 -0.07" rpy="0 1.57 0"/>
+		<origin xyz="0.51 -0.5 -0.02" rpy="0 1.57 0"/>
         <parent link="base_link"/>
         <child link="back_left_wheel"/>
 		<axis xyz="0 0 1"/>
-		<limit effort="30" velocity="2.0"/>
+		<limit effort="30" velocity="10.0"/>
+ 	</joint>
+	<joint name="mid_wheel_joint" type="continuous">
+		<origin xyz="0 0 -0.27" rpy="0 0 0"/>
+        <parent link="base_link"/>
+        <child link="mid_wheel"/>
  	</joint>
 	<joint name="front_panel_joint" type="prismatic">
@@ -253,5 +294,5 @@
 		<limit effort="10" velocity="1.0" lower="0" upper="0.25" />
  	</joint>
-	<joint name="mid_panel_prism_joint" type="prismatic">
+	<!-- <joint name="mid_panel_prism_joint" type="prismatic">
         <parent link="base_link"/>
         <child link="mid_panel_prism"/>
@@ -264,24 +305,24 @@
 		<axis xyz="1 0 0"/>
 		<limit effort="1.0" velocity="0.5" lower="0" upper="1.57" />
- 	</joint>
+ 	</joint> -->
 <!-- *********************** CONTROLEUR ******************************  -->
   	<gazebo>
-    <plugin name='diff_drive' filename='libgazebo_ros_diff_drive.so'>
-      <!-- wheels -->
-      <left_joint>front_left_joint</left_joint>
-      <right_joint>front_right_joint</right_joint>
-      <!-- kinematics -->
-      <wheel_separation>1.25</wheel_separation>
-      <wheel_diameter>0.6</wheel_diameter>
-      <!-- limits -->
-      <max_wheel_torque>20</max_wheel_torque>
-      <max_wheel_acceleration>1.0</max_wheel_acceleration>
-      <!-- output -->
-      <publish_odom>true</publish_odom>
-      <publish_odom_tf>true</publish_odom_tf>
-      <publish_wheel_tf>true</publish_wheel_tf>
-      <robot_base_frame>base_link</robot_base_frame>
-    </plugin>
-  </gazebo>
+		<plugin name='diff_drive' filename='libgazebo_ros_diff_drive.so'>
+		<!-- wheels -->
+		<left_joint>back_left_joint</left_joint>
+		<right_joint>back_right_joint</right_joint>
+		<!-- kinematics -->
+		<wheel_separation>1.25</wheel_separation>
+		<wheel_diameter>0.6</wheel_diameter>
+		<!-- limits -->
+		<max_wheel_torque>20</max_wheel_torque>
+		<max_wheel_acceleration>1.0</max_wheel_acceleration>
+		<!-- output -->
+		<publish_odom>true</publish_odom>
+		<publish_odom_tf>true</publish_odom_tf>
+		<publish_wheel_tf>true</publish_wheel_tf>
+		<robot_base_frame>base_link</robot_base_frame>
+		</plugin>
+  	</gazebo>
     <!-- <gazebo>
     <plugin name='diff_drive' filename='libgazebo_ros_diff_drive.so'>
