Commit message: New bot architecture

File: totem/bot/urdf/bot.urdf.xacro (robot description, xacro)
@@ -22,11 +22,4 @@
 		</inertial>
 	</xacro:macro>
-	<link name="base_footprint"/>
-	<!-- The base footprint of the robot is located underneath the chassis -->
-	<joint name="base_joint" type="fixed">
-		<parent link="base_link"/>
-		<child link="base_footprint" />
-		<origin xyz="0.0 0.0 -0.1" rpy="0 0 0"/>
-	</joint>
  	<link name="base_link">
 		<visual>
@@ -84,5 +77,5 @@
 			</geometry>
 		</collision>
-		<xacro:box_inertia m="35.0" w="3." d="2." h="1"/>
+		<xacro:box_inertia m="5.0" w="3." d="2." h="0.5"/>
   	</link>
 	<link name="back_left_wheel">
@@ -104,4 +97,13 @@
 		<xacro:cylinder_inertia m="2" r="0.25" h="0.2"/>
   	</link>
+	<gazebo reference="back_left_wheel">
+		<mu1>1.2</mu1>
+		<mu2>1.2</mu2>
+		<material>Gazebo/Blue</material>
+		<kp>500000.0</kp>
+		<kd>10.0</kd>
+		<minDepth>0.001</minDepth>
+		<maxVel>0.1</maxVel>
+  	</gazebo>
 	<link name="back_right_wheel">
   		<visual>
@@ -122,9 +124,18 @@
 		<xacro:cylinder_inertia m="2" r="0.25" h="0.1"/>
   	</link>
+	<gazebo reference="back_right_wheel">
+		<mu1>1.2</mu1>
+		<mu2>1.2</mu2>
+		<material>Gazebo/Blue</material>
+		<kp>500000.0</kp>
+		<kd>10.0</kd>
+		<minDepth>0.001</minDepth>
+		<maxVel>0.1</maxVel>
+  	</gazebo>
 	<link name="mid_wheel">
   		<visual>
 		    <origin xyz="0 0 0" rpy="0 0 0"/>
 			<geometry>
-				<sphere radius="0.02"/>
+				<sphere radius="0.05"/>
 			</geometry>
 			<material name="d">
@@ -135,62 +146,8 @@
 		    <origin xyz="0 0 0" rpy="0 0 0"/>
 			<geometry>
-				<sphere radius="0.02"/>
-			</geometry>
-		</collision>
-		<xacro:sphere_inertia m="1" r="0.02"/>
-  	</link>
-	<!-- <link name="front_left_wheel">
-  		<visual>
-		    <origin xyz="0 0 0" rpy="0 0 0"/>
-			<geometry>
-				<cylinder radius="0.25" length="0.1"/>
-			</geometry>
-			<material name="d">
-	       		<color rgba="0 0 0 0"/>
-	     	</material>
-		</visual>
-		<collision>
-		    <origin xyz="0 0 0" rpy="0 0 0"/>
-			<geometry>
-				<cylinder radius="0.25" length="0.1"/>
-			</geometry>
-		</collision>
-		<xacro:cylinder_inertia m="2" r="0.25" h="0.1"/>
-  	</link>
-	<link name="front_right_wheel">
-  		<visual>
-		    <origin xyz="0 0 0" rpy="0 0 0"/>
-			<geometry>
-				<cylinder radius="0.25" length="0.1"/>
-			</geometry>
-			<material name="d">
-	       		<color rgba="0 0 0 0"/>
-	     	</material>
-		</visual>
-		<collision>
-		    <origin xyz="0 0 0" rpy="0 0 0"/>
-			<geometry>
-				<cylinder radius="0.25" length="0.1"/>
-			</geometry>
-		</collision>
-		<xacro:cylinder_inertia m="2" r="0.25" h="0.1"/>
-  	</link> -->
-	<link name="front_panel">
-  		<visual>
-		    <origin xyz="0 0.7 0" rpy="0 0 0"/>
-			<geometry>
-				<box size="0.7 0.1 0.5"/>
-			</geometry>
-			<material name="f">
-	       		<color rgba="0 0 0.9 1.0"/>
-	     	</material>
-		</visual>
-		<collision>
-		    <origin xyz="0 0.7 0" rpy="0 0 0"/>
-			<geometry>
-				<box size="0.7 0.1 0.5"/>
-			</geometry>
-		</collision>
-		<xacro:box_inertia m="10.0" w="0.7" d="0.1" h="0.5"/>
+				<sphere radius="0.05"/>
+			</geometry>
+		</collision>
+		<xacro:sphere_inertia m="1" r="0.05"/>
   	</link>
 	<gazebo reference="mid_wheel">
@@ -203,72 +160,30 @@
 		<maxVel>0.1</maxVel>
 	</gazebo>
-	<!-- <link name="mid_panel">
-  		<visual>
-		    <origin xyz="0 0 0" rpy="0 0 0"/>
-			<geometry>
-				<box size="0.6 0.02 0.5"/>
-			</geometry>
-			<material name="l">
-	       		<color rgba="1 0 0 1.0"/>
-	     	</material>
-		</visual>
-		<collision>
-		    <origin xyz="0 0 0" rpy="0 0 0"/>
-			<geometry>
-				<box size="0.9 0.02 0.5"/>
-			</geometry>
-		</collision>
-		<xacro:box_inertia m="10.0" w="0.9" d="0.02" h="1"/>
-  	</link>
-	<link name="mid_panel_prism">
-  		<visual>
-		    <origin xyz="-0.335 0 0" rpy="0 0 0"/>
-			<geometry>
-				<box size="0.05 0.1 0.1"/>
-			</geometry>
-			<material name="m">
-	       		<color rgba="1 1 0 1.0"/>
-	     	</material>
-		</visual>
-		<xacro:box_inertia m="0" w="0.05" d="0.1" h="0.1"/>
-  	</link> -->
+	<link name="front_panel">
+  		<visual>
+		    <origin xyz="0 0.7 0" rpy="0 0 0"/>
+			<geometry>
+				<box size="0.7 0.1 0.5"/>
+			</geometry>
+			<material name="f">
+	       		<color rgba="0 0 0.9 1.0"/>
+	     	</material>
+		</visual>
+		<collision>
+		    <origin xyz="0 0.7 0" rpy="0 0 0"/>
+			<geometry>
+				<box size="0.7 0.1 0.5"/>
+			</geometry>
+		</collision>
+		<xacro:box_inertia m="1.0" w="0.7" d="0.1" h="0.5"/>
+  	</link>
 	<gazebo reference="base_link">
 		<material>Gazebo/Red</material>
 	</gazebo>
-	<!-- <gazebo reference="front_right_wheel">
-		<material>Gazebo/Blue</material>
-	</gazebo>
-	<gazebo reference="front_left_wheel">
-		<material>Gazebo/Blue</material>
-	</gazebo> -->
-	<gazebo reference="back_right_wheel">
-		<material>Gazebo/Blue</material>
-	</gazebo>
-	<gazebo reference="back_left_wheel">
-		<material>Gazebo/Blue</material>
-	</gazebo>
-	<!-- <gazebo reference="mid_panel">
-		<material>Gazebo/Blue</material>
-	</gazebo> -->
 	<gazebo reference="front_panel">
 		<material>Gazebo/Red</material>
 	</gazebo>
-	<!-- <joint name="front_right_joint" type="continuous">
-		<origin xyz="-0.51 0.5 -0.07" rpy="0 1.57 0"/>
-        <parent link="base_link"/>
-        <child link="front_right_wheel"/>
-		<limit effort="30" velocity="2.0"/>
-      	<axis xyz="0 0 1" />
-      	<dynamics damping="1.0" />
- 	</joint>
-	<joint name="front_left_joint" type="continuous">
-		<origin xyz="0.51 0.5 -0.07" rpy="0 1.57 0"/>
-        <parent link="base_link"/>
-        <child link="front_left_wheel"/>
-		<axis xyz="0 0 1"/>
-		<limit effort="30" velocity="2.0"/>
- 	</joint> -->
 	<joint name="back_right_joint" type="continuous">
-		<origin xyz="-0.51 -0.5 -0.02" rpy="0 1.57 0"/>
+		<origin xyz="-0.51 -0.5 -0.05" rpy="0 1.57 0"/>
         <parent link="base_link"/>
         <child link="back_right_wheel"/>
@@ -277,5 +192,5 @@
  	</joint>
 	<joint name="back_left_joint" type="continuous">
-		<origin xyz="0.51 -0.5 -0.02" rpy="0 1.57 0"/>
+		<origin xyz="0.51 -0.5 -0.05" rpy="0 1.57 0"/>
         <parent link="base_link"/>
         <child link="back_left_wheel"/>
@@ -284,5 +199,5 @@
  	</joint>
 	<joint name="mid_wheel_joint" type="continuous">
-		<origin xyz="0 0 -0.27" rpy="0 0 0"/>
+		<origin xyz="0 0 -0.25" rpy="0 0 0"/>
         <parent link="base_link"/>
         <child link="mid_wheel"/>
@@ -294,48 +209,32 @@
 		<limit effort="10" velocity="1.0" lower="0" upper="0.25" />
  	</joint>
-	<!-- <joint name="mid_panel_prism_joint" type="prismatic">
-        <parent link="base_link"/>
-        <child link="mid_panel_prism"/>
-		<axis xyz="0 1 0"/>
-		<limit effort="1.0" velocity="0.5" lower="0" upper="0.1" />
- 	</joint>
-	<joint name="mid_panel_joint" type="revolute">
-        <parent link="mid_panel_prism"/>
-        <child link="mid_panel"/>
-		<axis xyz="1 0 0"/>
-		<limit effort="1.0" velocity="0.5" lower="0" upper="1.57" />
- 	</joint> -->
 <!-- *********************** CONTROLEUR ******************************  -->
   	<gazebo>
 		<plugin name='diff_drive' filename='libgazebo_ros_diff_drive.so'>
-		<!-- wheels -->
-		<left_joint>back_left_joint</left_joint>
-		<right_joint>back_right_joint</right_joint>
-		<!-- kinematics -->
-		<wheel_separation>1.25</wheel_separation>
-		<wheel_diameter>0.6</wheel_diameter>
-		<!-- limits -->
-		<max_wheel_torque>20</max_wheel_torque>
-		<max_wheel_acceleration>1.0</max_wheel_acceleration>
-		<!-- output -->
-		<publish_odom>true</publish_odom>
-		<publish_odom_tf>true</publish_odom_tf>
-		<publish_wheel_tf>true</publish_wheel_tf>
-		<robot_base_frame>base_link</robot_base_frame>
+			<!-- wheels -->
+			<left_joint>back_left_joint</left_joint>
+			<right_joint>back_right_joint</right_joint>
+			<!-- kinematics -->
+			<wheel_separation>1.6</wheel_separation>
+			<wheel_diameter>0.5</wheel_diameter>
+			<!-- limits -->
+			<max_wheel_torque>20</max_wheel_torque>
+			<max_wheel_acceleration>1.0</max_wheel_acceleration>
+			<!-- output -->
+			<publish_odom>true</publish_odom>
+			<publish_odom_tf>true</publish_odom_tf>
+			<publish_wheel_tf>true</publish_wheel_tf>
+			<robot_base_frame>base_link</robot_base_frame>
 		</plugin>
   	</gazebo>
-    <!-- <gazebo>
-    <plugin name='diff_drive' filename='libgazebo_ros_diff_drive.so'>
-      <left_joint>back_left_joint</left_joint>
-      <right_joint>back_right_joint</right_joint>
-      <wheel_separation>1.25</wheel_separation>
-      <wheel_diameter>0.6</wheel_diameter>
-      <max_wheel_torque>20</max_wheel_torque>
-      <max_wheel_acceleration>1.0</max_wheel_acceleration>
-      <publish_odom>true</publish_odom>
-      <publish_odom_tf>true</publish_odom_tf>
-      <publish_wheel_tf>true</publish_wheel_tf>
-      <robot_base_frame>base_link</robot_base_frame>
-    </plugin>
-  </gazebo> -->
+	<gazebo>
+		<plugin name="imu_plugin" filename="libgazebo_ros_imu.so">
+		<alwaysOn>true</alwaysOn>
+		<bodyName>base_footprint</bodyName>
+		<topicName>imu</topicName>
+		<serviceName>imu_service</serviceName>
+		<gaussianNoise>0.0</gaussianNoise>
+		<updateRate>20.0</updateRate>
+		</plugin>
+  	</gazebo>
 </robot>

Commit message: robot velocity command direction fixed

File: totem/bot/urdf/bot.urdf.xacro (robot description, xacro)
@@ -24,7 +24,7 @@
  	<link name="base_link">
 		<visual>
-		    <origin xyz="0.4 0 0" rpy="0 0 0"/>
-			<geometry>
-				<box size="0.1 1.5 0.5"/>
+		    <origin xyz="0 0.4 0" rpy="0 0 0"/>
+			<geometry>
+				<box size="1.5 0.1 0.5"/>
 			</geometry>
 			<material name="c1">
@@ -33,7 +33,7 @@
 		</visual>
   		<visual>
-		    <origin xyz="-0.4 0 0" rpy="0 0 0"/>
-			<geometry>
-				<box size="0.1 1.5 0.5"/>
+		    <origin xyz="0 -0.4 0" rpy="0 0 0"/>
+			<geometry>
+				<box size="1.5 0.1 0.5"/>
 			</geometry>
 			<material name="c">
@@ -42,7 +42,7 @@
 		</visual>
   		<visual>
-		    <origin xyz="0 -0.7 0" rpy="0 0 0"/>
-			<geometry>
-				<box size="0.7 0.1 0.5"/>
+		    <origin xyz="0.7 0 0" rpy="0 0 0"/>
+			<geometry>
+				<box size="0.1 0.7 0.5"/>
 			</geometry>
 			<material name="c2">
@@ -51,7 +51,7 @@
 		</visual>
   		<visual>
-          	<origin xyz="0 -0.2 0" rpy="0 0 0"/>
-			<geometry>
-				<box size="0.7 0.95 0.5"/>
+          	<origin xyz="0.2 0 0" rpy="0 0 0"/>
+			<geometry>
+				<box size="0.95 0.7 0.5"/>
 			</geometry>
 			<material name="c">
@@ -60,19 +60,25 @@
 		</visual>
 		<collision>
-		    <origin xyz="0 -0.7 0" rpy="0 0 0"/>
-			<geometry>
-				<box size="0.7 0.1 0.5"/>
-			</geometry>
-		</collision>
-		<collision>
-		    <origin xyz="0.4  0 0" rpy="0 0 0"/>
-			<geometry>
-				<box size="0.1 1.5 0.5"/>
-			</geometry>
-		</collision>
-		<collision>
-		    <origin xyz="-0.4 0 0" rpy="0 0 0"/>
-			<geometry>
-				<box size="0.1 1.5 0.5"/>
+		    <origin xyz="-0.7 0 0" rpy="0 0 0"/>
+			<geometry>
+				<box size="0.1 0.7 0.5"/>
+			</geometry>
+		</collision>
+		<collision>
+		    <origin xyz="0 0.4 0" rpy="0 0 0"/>
+			<geometry>
+				<box size="1.5 0.1 0.5"/>
+			</geometry>
+		</collision>
+		<collision>
+		    <origin xyz="0 -0.4 0" rpy="0 0 0"/>
+			<geometry>
+				<box size="1.5 0.1 0.5"/>
+			</geometry>
+		</collision>
+		<collision>
+			<origin xyz="0.2 0 0" rpy="0 0 0"/>
+			<geometry>
+				<box size="0.95 0.7 0.5"/>
 			</geometry>
 		</collision>
@@ -162,7 +168,7 @@
 	<link name="front_panel">
   		<visual>
-		    <origin xyz="0 0.7 0" rpy="0 0 0"/>
-			<geometry>
-				<box size="0.7 0.1 0.5"/>
+		    <origin xyz="-0.7 0 0" rpy="0 0 0"/>
+			<geometry>
+				<box size="0.1 0.7 0.5"/>
 			</geometry>
 			<material name="f">
@@ -171,7 +177,7 @@
 		</visual>
 		<collision>
-		    <origin xyz="0 0.7 0" rpy="0 0 0"/>
-			<geometry>
-				<box size="0.7 0.1 0.5"/>
+		    <origin xyz="-0.7 0 0" rpy="0 0 0"/>
+			<geometry>
+				<box size="0.1 0.7 0.5"/>
 			</geometry>
 		</collision>
@@ -185,5 +191,5 @@
 	</gazebo>
 	<joint name="back_right_joint" type="continuous">
-		<origin xyz="-0.51 -0.5 -0.05" rpy="0 1.57 0"/>
+		<origin xyz="0.5 -0.51 -0.05" rpy="1.57 0 0"/>
         <parent link="base_link"/>
         <child link="back_right_wheel"/>
@@ -192,5 +198,5 @@
  	</joint>
 	<joint name="back_left_joint" type="continuous">
-		<origin xyz="0.51 -0.5 -0.05" rpy="0 1.57 0"/>
+		<origin xyz="0.5 0.51 -0.05" rpy="1.57 0 0"/>
         <parent link="base_link"/>
         <child link="back_left_wheel"/>
@@ -231,5 +237,5 @@
 		<plugin name="imu_plugin" filename="libgazebo_ros_imu.so">
 		<alwaysOn>true</alwaysOn>
-		<bodyName>base_footprint</bodyName>
+		<bodyName>base_link</bodyName>
 		<topicName>imu</topicName>
 		<serviceName>imu_service</serviceName>
